Commit message: added base link mesh stl file and scaling in urdf model

File: qbot_nodes_cpp/urdf/qbot_description.urdf (robot description, URDF)
Before this commit: robot qbot, 3 links, 2 joints
Links:
- link base_link: geometry visual mesh filename=package://qbot_nodes_cpp/meshes/rover_base.stl scale=${dim_scale} ${dim_scale} ${dim_scale}
