Commit message: added sensor to urdf

File: qbot_nodes_cpp/urdf/qbot_description_no_xacro.urdf (robot description, URDF)
Before this commit: robot qbot, 5 links, 4 joints
Links:
- added link base_laser; visual box size=1.0 2.0 1.0
Joints:
- added joint base_to_laser: type fixed, parent base_link, child base_laser, origin xyz=0.105 0 0.22 rpy=0 0 0

Commit message: correct base laser origin in urdf

File: qbot_nodes_cpp/urdf/qbot_description_no_xacro.urdf (robot description, URDF)
Before this commit: robot qbot, 6 links, 5 joints
Joints:
- joint base_to_laser: origin xyz=0.105 0 0.22 rpy=0 0 0 -> xyz=5.0 0 2.0 rpy=0 0 0
